File: Atrix_breakout.sch (EAGLE design)
At the start: 8 parts

Commit message: Update README with How-to
Parts:
- removed 14: (no value), wirepad:1,6/0,8
- added AL, GND1: (no value), wirepad:1,6/0,8
Connections:
- removed net N$5: 14.P, U$1.14
- new net N$2: AL.P, U$1.ACC_INDICATOR
- net N$1: now also GND1.P
Other:
- moved on the sheet: GND
Changed lines of the file:
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@@
 <part name="D-" library="wirepad" deviceset="1,6/0,8" device=""/>
 <part name="D+" library="wirepad" deviceset="1,6/0,8" device=""/>
-<part name="14" library="wirepad" deviceset="1,6/0,8" device=""/>
 <part name="RX" library="wirepad" deviceset="1,6/0,8" device=""/>
 <part name="TX" library="wirepad" deviceset="1,6/0,8" device=""/>
 <part name="5V" library="wirepad" deviceset="1,6/0,8" device=""/>
+<part name="AL" library="wirepad" deviceset="1,6/0,8" device=""/>
+<part name="GND1" library="wirepad" deviceset="1,6/0,8" device=""/>
 </parts>
 <sheets>
@@
 <instances>
 <instance part="U$1" gate="G$1" x="134.62" y="45.72"/>
-<instance part="GND" gate="P" x="114.3" y="81.28" smashed="yes">
-<attribute name="NAME" x="105.537" y="80.5942" size="1.778" layer="95"/>
-<attribute name="VALUE" x="113.157" y="77.978" size="1.778" layer="96"/>
+<instance part="GND" gate="P" x="101.6" y="81.28" smashed="yes">
+<attribute name="NAME" x="92.837" y="80.5942" size="1.778" layer="95"/>
+<attribute name="VALUE" x="100.457" y="77.978" size="1.778" layer="96"/>
 </instance>
 <instance part="D-" gate="P" x="114.3" y="20.32" smashed="yes">
@@
 <attribute name="NAME" x="108.077" y="14.5542" size="1.778" layer="95"/>
 <attribute name="VALUE" x="113.157" y="11.938" size="1.778" layer="96"/>
-</instance>
-<instance part="14" gate="P" x="114.3" y="48.26" smashed="yes">
-<attribute name="NAME" x="108.077" y="47.5742" size="1.778" layer="95"/>
-<attribute name="VALUE" x="113.157" y="44.958" size="1.778" layer="96"/>
 </instance>
 <instance part="RX" gate="P" x="114.3" y="50.8" smashed="yes">
@@
 <attribute name="VALUE" x="113.157" y="22.098" size="1.778" layer="96"/>
 </instance>
+<instance part="AL" gate="P" x="114.3" y="30.48" smashed="yes">
+<attribute name="NAME" x="108.077" y="29.7942" size="1.778" layer="95"/>
+<attribute name="VALUE" x="113.157" y="27.178" size="1.778" layer="96"/>
+</instance>
+<instance part="GND1" gate="P" x="101.6" y="83.82" smashed="yes">
+<attribute name="NAME" x="92.837" y="83.1342" size="1.778" layer="95"/>
+<attribute name="VALUE" x="100.457" y="80.518" size="1.778" layer="96"/>
+</instance>
 </instances>
 <busses>
@@
 <pinref part="U$1" gate="G$1" pin="GND@1"/>
 <pinref part="GND" gate="P" pin="P"/>
+<wire x1="104.14" y1="81.28" x2="106.68" y2="81.28" width="0.1524" layer="91"/>
+<wire x1="106.68" y1="81.28" x2="116.84" y2="81.28" width="0.1524" layer="91"/>
+<wire x1="106.68" y1="81.28" x2="106.68" y2="83.82" width="0.1524" layer="91"/>
+<junction x="106.68" y="81.28"/>
+<pinref part="GND1" gate="P" pin="P"/>
+<wire x1="106.68" y1="83.82" x2="104.14" y2="83.82" width="0.1524" layer="91"/>
 </segment>
 </net>
@@
 <pinref part="U$1" gate="G$1" pin="USB_D+"/>
 <pinref part="D+" gate="P" pin="P"/>
-</segment>
-</net>
-<net name="N$5" class="0">
-<segment>
-<pinref part="U$1" gate="G$1" pin="14"/>
-<pinref part="14" gate="P" pin="P"/>
 </segment>
 </net>
@@
 </segment>
 </net>
+<net name="N$2" class="0">
+<segment>
+<pinref part="U$1" gate="G$1" pin="ACC_INDICATOR"/>
+<pinref part="AL" gate="P" pin="P"/>
+</segment>
+</net>

Commit message: updates
Connections:
- net N$1 renamed GND
Other:
- moved on the sheet: GND, GND1
Changed lines of the file:
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@@
 <instances>
 <instance part="U$1" gate="G$1" x="134.62" y="45.72"/>
-<instance part="GND" gate="P" x="101.6" y="81.28" smashed="yes">
-<attribute name="NAME" x="92.837" y="80.5942" size="1.778" layer="95"/>
-<attribute name="VALUE" x="100.457" y="77.978" size="1.778" layer="96"/>
+<instance part="GND" gate="P" x="93.98" y="78.74" smashed="yes">
+<attribute name="NAME" x="85.217" y="78.0542" size="1.778" layer="95"/>
+<attribute name="VALUE" x="92.837" y="75.438" size="1.778" layer="96"/>
 </instance>
 <instance part="D-" gate="P" x="114.3" y="20.32" smashed="yes">
@@
 <attribute name="VALUE" x="113.157" y="27.178" size="1.778" layer="96"/>
 </instance>
-<instance part="GND1" gate="P" x="101.6" y="83.82" smashed="yes">
-<attribute name="NAME" x="92.837" y="83.1342" size="1.778" layer="95"/>
-<attribute name="VALUE" x="100.457" y="80.518" size="1.778" layer="96"/>
+<instance part="GND1" gate="P" x="93.98" y="81.28" smashed="yes">
+<attribute name="NAME" x="85.217" y="80.5942" size="1.778" layer="95"/>
+<attribute name="VALUE" x="92.837" y="77.978" size="1.778" layer="96"/>
 </instance>
 </instances>
@@
 </busses>
 <nets>
-<net name="N$1" class="0">
-<segment>
-<pinref part="U$1" gate="G$1" pin="GND@1"/>
-<pinref part="GND" gate="P" pin="P"/>
-<wire x1="104.14" y1="81.28" x2="106.68" y2="81.28" width="0.1524" layer="91"/>
-<wire x1="106.68" y1="81.28" x2="116.84" y2="81.28" width="0.1524" layer="91"/>
-<wire x1="106.68" y1="81.28" x2="106.68" y2="83.82" width="0.1524" layer="91"/>
-<junction x="106.68" y="81.28"/>
-<pinref part="GND1" gate="P" pin="P"/>
-<wire x1="106.68" y1="83.82" x2="104.14" y2="83.82" width="0.1524" layer="91"/>
-</segment>
-</net>
 <net name="N$3" class="0">
 <segment>
@@
 </segment>
 </net>
+<net name="GND" class="0">
+<segment>
+<pinref part="U$1" gate="G$1" pin="GND@1"/>
+<wire x1="116.84" y1="81.28" x2="114.3" y2="81.28" width="0.1524" layer="91"/>
+<label x="111.76" y="81.28" size="1.778" layer="95"/>
+</segment>
+<segment>
+<pinref part="GND1" gate="P" pin="P"/>
+<wire x1="96.52" y1="81.28" x2="99.06" y2="81.28" width="0.1524" layer="91"/>
+<label x="99.06" y="81.28" size="1.778" layer="95"/>
+</segment>
+<segment>
+<pinref part="GND" gate="P" pin="P"/>
+<wire x1="96.52" y1="78.74" x2="99.06" y2="78.74" width="0.1524" layer="91"/>
+<label x="99.06" y="78.74" size="1.778" layer="95"/>
+</segment>
+</net>

Commit message: Correct AL pin name, should be ACC
Parts:
- renumbered AL to ACC
Changed lines of the file:
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@@
 <part name="TX" library="wirepad" deviceset="1,6/0,8" device=""/>
 <part name="5V" library="wirepad" deviceset="1,6/0,8" device=""/>
-<part name="AL" library="wirepad" deviceset="1,6/0,8" device=""/>
+<part name="ACC" library="wirepad" deviceset="1,6/0,8" device=""/>
 <part name="GND1" library="wirepad" deviceset="1,6/0,8" device=""/>
 </parts>
@@
 <attribute name="VALUE" x="113.157" y="22.098" size="1.778" layer="96"/>
 </instance>
-<instance part="AL" gate="P" x="114.3" y="30.48" smashed="yes">
+<instance part="ACC" gate="P" x="114.3" y="30.48" smashed="yes">
 <attribute name="NAME" x="108.077" y="29.7942" size="1.778" layer="95"/>
 <attribute name="VALUE" x="113.157" y="27.178" size="1.778" layer="96"/>
@@
 <segment>
 <pinref part="U$1" gate="G$1" pin="ACC_INDICATOR"/>
-<pinref part="AL" gate="P" pin="P"/>
+<pinref part="ACC" gate="P" pin="P"/>
 </segment>
 </net>

Commit message: Push to OpenJB
Parts:
- removed 5V, D+, D-, GND1, RX, TX: (no value), wirepad:1,6/0,8
- added JP1: FTDI, SparkFun-Connectors:FTDI_BASICPTH
- added X1: USB-MICROB, Pinoccio:USB-MICROB
- ACC, GND: device wirepad:1,6/0,8 -> wirepad:1,6/0,9
Connections:
- removed net N$3: D-.P, U$1.USB_D-
- removed net N$4: D+.P, U$1.USB_D+
- removed net N$6: RX.P, U$1.RX
- removed net N$7: TX.P, U$1.TX
- removed net N$8: 5V.P, U$1.USB_5V
- new net 5V: U$1.USB_5V, X1.VBUS
- new net D+: U$1.USB_D+, X1.D+
- new net D-: U$1.USB_D-, X1.D-
- new net RX: JP1.3, U$1.RX
- new net TX: JP1.2, U$1.TX
- net GND: now also JP1.6, X1.GND; no longer GND1.P
Changed lines of the file:
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@@
 <parts>
 <part name="U$1" library="SparkFun-Connectors" deviceset="IPOD_CONNECTOR_MALE" device=""/>
-<part name="GND" library="wirepad" deviceset="1,6/0,8" device=""/>
-<part name="D-" library="wirepad" deviceset="1,6/0,8" device=""/>
-<part name="D+" library="wirepad" deviceset="1,6/0,8" device=""/>
-<part name="RX" library="wirepad" deviceset="1,6/0,8" device=""/>
-<part name="TX" library="wirepad" deviceset="1,6/0,8" device=""/>
-<part name="5V" library="wirepad" deviceset="1,6/0,8" device=""/>
-<part name="ACC" library="wirepad" deviceset="1,6/0,8" device=""/>
-<part name="GND1" library="wirepad" deviceset="1,6/0,8" device=""/>
+<part name="JP1" library="SparkFun-Connectors" deviceset="FTDI_BASIC" device="PTH" value="FTDI"/>
+<part name="X1" library="Pinoccio" deviceset="USB" device="-MICROB" value="USB-MICROB"/>
+<part name="GND" library="wirepad" deviceset="1,6/0,9" device=""/>
+<part name="ACC" library="wirepad" deviceset="1,6/0,9" device=""/>
 </parts>
 <sheets>
@@
 <instances>
 <instance part="U$1" gate="G$1" x="134.62" y="45.72"/>
-<instance part="GND" gate="P" x="93.98" y="78.74" smashed="yes">
-<attribute name="NAME" x="85.217" y="78.0542" size="1.778" layer="95"/>
-<attribute name="VALUE" x="92.837" y="75.438" size="1.778" layer="96"/>
-</instance>
-<instance part="D-" gate="P" x="114.3" y="20.32" smashed="yes">
-<attribute name="NAME" x="108.077" y="19.6342" size="1.778" layer="95"/>
-<attribute name="VALUE" x="113.157" y="17.018" size="1.778" layer="96"/>
-</instance>
-<instance part="D+" gate="P" x="114.3" y="15.24" smashed="yes">
-<attribute name="NAME" x="108.077" y="14.5542" size="1.778" layer="95"/>
-<attribute name="VALUE" x="113.157" y="11.938" size="1.778" layer="96"/>
-</instance>
-<instance part="RX" gate="P" x="114.3" y="50.8" smashed="yes">
-<attribute name="NAME" x="108.077" y="50.1142" size="1.778" layer="95"/>
-<attribute name="VALUE" x="113.157" y="47.498" size="1.778" layer="96"/>
-</instance>
-<instance part="TX" gate="P" x="114.3" y="53.34" smashed="yes">
-<attribute name="NAME" x="108.077" y="52.6542" size="1.778" layer="95"/>
-<attribute name="VALUE" x="113.157" y="50.038" size="1.778" layer="96"/>
-</instance>
-<instance part="5V" gate="P" x="114.3" y="25.4" smashed="yes">
-<attribute name="NAME" x="108.077" y="24.7142" size="1.778" layer="95"/>
-<attribute name="VALUE" x="113.157" y="22.098" size="1.778" layer="96"/>
-</instance>
-<instance part="ACC" gate="P" x="114.3" y="30.48" smashed="yes">
-<attribute name="NAME" x="108.077" y="29.7942" size="1.778" layer="95"/>
-<attribute name="VALUE" x="113.157" y="27.178" size="1.778" layer="96"/>
-</instance>
-<instance part="GND1" gate="P" x="93.98" y="81.28" smashed="yes">
-<attribute name="NAME" x="85.217" y="80.5942" size="1.778" layer="95"/>
-<attribute name="VALUE" x="92.837" y="77.978" size="1.778" layer="96"/>
-</instance>
+<instance part="JP1" gate="G$1" x="58.42" y="66.04"/>
+<instance part="X1" gate="G$1" x="58.42" y="50.8" smashed="yes" rot="R180"/>
+<instance part="GND" gate="1" x="101.6" y="30.48" rot="R180"/>
+<instance part="ACC" gate="1" x="111.76" y="30.48"/>
 </instances>
 <busses>
 </busses>
 <nets>
-<net name="N$3" class="0">
-<segment>
-<pinref part="U$1" gate="G$1" pin="USB_D-"/>
-<pinref part="D-" gate="P" pin="P"/>
-</segment>
-</net>
-<net name="N$4" class="0">
-<segment>
-<pinref part="U$1" gate="G$1" pin="USB_D+"/>
-<pinref part="D+" gate="P" pin="P"/>
-</segment>
-</net>
-<net name="N$6" class="0">
-<segment>
-<pinref part="U$1" gate="G$1" pin="RX"/>
-<pinref part="RX" gate="P" pin="P"/>
-</segment>
-</net>
-<net name="N$7" class="0">
-<segment>
-<pinref part="U$1" gate="G$1" pin="TX"/>
-<pinref part="TX" gate="P" pin="P"/>
-</segment>
-</net>
-<net name="N$8" class="0">
-<segment>
-<pinref part="U$1" gate="G$1" pin="USB_5V"/>
-<pinref part="5V" gate="P" pin="P"/>
-</segment>
-</net>
-<net name="N$2" class="0">
-<segment>
-<pinref part="U$1" gate="G$1" pin="ACC_INDICATOR"/>
-<pinref part="ACC" gate="P" pin="P"/>
-</segment>
-</net>
 <net name="GND" class="0">
 <segment>
@@
 </segment>
 <segment>
-<pinref part="GND1" gate="P" pin="P"/>
-<wire x1="96.52" y1="81.28" x2="99.06" y2="81.28" width="0.1524" layer="91"/>
-<label x="99.06" y="81.28" size="1.778" layer="95"/>
+<pinref part="JP1" gate="G$1" pin="6"/>
+<wire x1="63.5" y1="73.66" x2="66.04" y2="73.66" width="0.1524" layer="91"/>
+<label x="66.04" y="73.66" size="1.778" layer="95"/>
 </segment>
 <segment>
-<pinref part="GND" gate="P" pin="P"/>
-<wire x1="96.52" y1="78.74" x2="99.06" y2="78.74" width="0.1524" layer="91"/>
-<label x="99.06" y="78.74" size="1.778" layer="95"/>
+<pinref part="X1" gate="G$1" pin="GND"/>
+<wire x1="60.96" y1="50.8" x2="63.5" y2="50.8" width="0.1524" layer="91"/>
+<label x="66.04" y="50.8" size="1.778" layer="95"/>
+</segment>
+<segment>
+<wire x1="99.06" y1="30.48" x2="96.52" y2="30.48" width="0.1524" layer="91"/>
+<label x="91.44" y="30.48" size="1.778" layer="95"/>
+<pinref part="GND" gate="1" pin="P"/>
 </segment>
 </net>
+<net name="RX" class="0">
+<segment>
+<pinref part="JP1" gate="G$1" pin="3"/>
+<wire x1="63.5" y1="66.04" x2="66.04" y2="66.04" width="0.1524" layer="91"/>
+<label x="66.04" y="66.04" size="1.778" layer="95"/>
+</segment>
+<segment>
+<pinref part="U$1" gate="G$1" pin="RX"/>
+<wire x1="116.84" y1="50.8" x2="114.3" y2="50.8" width="0.1524" layer="91"/>
+<label x="111.76" y="50.8" size="1.778" layer="95"/>
+</segment>
+</net>
+<net name="TX" class="0">
+<segment>
+<pinref part="U$1" gate="G$1" pin="TX"/>
+<wire x1="116.84" y1="53.34" x2="114.3" y2="53.34" width="0.1524" layer="91"/>
+<label x="111.76" y="53.34" size="1.778" layer="95"/>
+</segment>
+<segment>
+<pinref part="JP1" gate="G$1" pin="2"/>
+<wire x1="63.5" y1="63.5" x2="66.04" y2="63.5" width="0.1524" layer="91"/>
+<label x="66.04" y="63.5" size="1.778" layer="95"/>
+</segment>
+</net>
+<net name="D+" class="0">
+<segment>
+<pinref part="U$1" gate="G$1" pin="USB_D+"/>
+<wire x1="116.84" y1="15.24" x2="114.3" y2="15.24" width="0.1524" layer="91"/>
+<label x="111.76" y="15.24" size="1.778" layer="95"/>
+</segment>
+<segment>
+<pinref part="X1" gate="G$1" pin="D+"/>
+<wire x1="60.96" y1="43.18" x2="63.5" y2="43.18" width="0.1524" layer="91"/>
+<label x="63.5" y="43.18" size="1.778" layer="95"/>
+</segment>
+</net>
+<net name="D-" class="0">
+<segment>
+<pinref part="U$1" gate="G$1" pin="USB_D-"/>
+<wire x1="116.84" y1="20.32" x2="114.3" y2="20.32" width="0.1524" layer="91"/>
+<label x="111.76" y="20.32" size="1.778" layer="95"/>
+</segment>
+<segment>
+<pinref part="X1" gate="G$1" pin="D-"/>
+<wire x1="60.96" y1="45.72" x2="63.5" y2="45.72" width="0.1524" layer="91"/>
+<label x="63.5" y="45.72" size="1.778" layer="95"/>
+</segment>
+</net>
+<net name="5V" class="0">
+<segment>
+<pinref part="U$1" gate="G$1" pin="USB_5V"/>
+<wire x1="116.84" y1="25.4" x2="114.3" y2="25.4" width="0.1524" layer="91"/>
+<label x="111.76" y="25.4" size="1.778" layer="95"/>
+</segment>
+<segment>
+<pinref part="X1" gate="G$1" pin="VBUS"/>
+<wire x1="60.96" y1="48.26" x2="63.5" y2="48.26" width="0.1524" layer="91"/>
+<label x="66.04" y="48.26" size="1.778" layer="95"/>
+</segment>
+</net>
+<net name="N$1" class="0">
+<segment>
+<pinref part="U$1" gate="G$1" pin="ACC_INDICATOR"/>
+<wire x1="116.84" y1="30.48" x2="114.3" y2="30.48" width="0.1524" layer="91"/>
+<pinref part="ACC" gate="1" pin="P"/>
+</segment>
+</net>
